File: RGBClock.brd (EAGLE design)
At the start: 101.3 x 56.5 mm, 31 parts, among them K1 PIN20X2

Commit message: Finished board
Parts:
- removed D1, D2: LED-RGB-CA-THRUDIFFUSE, SparkFun-LED:LED-RGB-THRU
- removed R10, R11, R12, R13, R14, R15, R16, R17, R18, R7, R8, R9: (no value), SparkFun-Passives:0805
- added LED1, LED2: RGBLED_CA-5MM, adafruit:LED5MMRGB
- moved R1 4.41 mm to (85.3, 29.1)
- moved R2 4.34 mm to (61.6, 29.3)
- moved R3 4.20 mm to (8.15, 29.3)
- moved R6 4.15 mm to (31.5, 29.4)
- moved U$6 1.27 mm to (90.4, 25.1)
- moved K1 1.27 mm to (33.8, 52.5)
- moved U$3 1.27 mm to (55.5, 7.62)
- moved U$5 1.27 mm to (1.91, 7.62)
- moved U$4 1.27 mm to (25.4, 7.62)
- moved U$9 1.27 mm to (13.7, 25.3)
- moved BAT1 1.27 mm to (92.1, 49.5)
- moved R4 1.27 mm to (72.0, 53.7)
- moved R5 1.27 mm to (70.0, 53.7)
- moved RTC1 1.27 mm to (77.5, 52.8)
- moved U$2 1.27 mm to (79.0, 7.62)
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Connections:
- removed net N$6: D1.4, D2.4, U$8.46
- new net N$3: LED1.4, LED2.4, U$8.46
- net +3V3: now also U$6.31, U$7.31, U$8.31, U$9.31; no longer R10.2, R11.2, R12.2, R13.2, R14.2, R15.2, R16.2, R17.2, R18.2, R7.2, R8.2, R9.2
- net +5V: now also LED1.2, LED2.2, U$2.17, U$3.17, U$4.17, U$5.17
- net /BOE: no longer R12.1, R15.1, R18.1, R9.1
- net /GOE: no longer R11.1, R14.1, R17.1, R8.1
- net /ROE: no longer R10.1, R13.1, R16.1, R7.1
- net N$2: now also LED1.1, LED2.1; no longer D1.1, D2.1
- net N$5: now also LED1.3, LED2.3; no longer D1.3, D2.3
Routing:
- net +5V: track 0.00 -> 164.5 mm
- net LATCH: track 0.00 -> 135.6 mm, vias 0 -> 5
- net /GOE: track 22.7 -> 141.2 mm, vias 0 -> 5
- net /BOE: track 21.5 -> 139.2 mm, vias 0 -> 5
- net /ROE: track 24.9 -> 123.8 mm, vias 0 -> 5
- net DATA: track 7.55 -> 104.6 mm
- net GND: track 0.00 -> 49.2 mm, vias 0 -> 5
- net N$3: track 0.00 -> 47.2 mm
- net N$6: track 38.9 -> 0.00 mm
- net +3V3: track 0.00 -> 16.6 mm
- net CLK: track 117.4 -> 133.7 mm, vias 4 -> 5
- net N$5: track 36.4 -> 46.0 mm
- net N$2: track 32.0 -> 41.0 mm
- net N$15: track 38.9 -> 32.5 mm
- net N$8: track 2.90 -> 4.47 mm
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- added copper zone on layer 1, net +3V3
- added copper zone on layer 16, net GND

Commit message: Board, gerbers, and BOM
Parts:
- added C1: (no value), SparkFun-Passives:0805
Connections:
- net +3V3: now also C1.1
- net GND: now also C1.2
Routing:
- net GND: track 49.2 -> 58.1 mm
Changed lines of the file:
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@@
 <hole x="62.77" y="52.5" drill="2.75"/>
 <hole x="62.77" y="3.5" drill="2.75"/>
-<dimension x1="1.27" y1="53.5" x2="102.54" y2="53.5" x3="51.905" y3="63.5" textsize="1.778" layer="90"/>
-<dimension x1="4.27" y1="56.5" x2="3.81" y2="0" x3="-7.39958125" y3="28.343134375" textsize="1.778" layer="90"/>
 </plain>
 <attributes>
@@
 </class>
 </classes>
-<designrules name="default">
+<designrules name="default *">
 <description language="de">&lt;b&gt;EAGLE Design Rules&lt;/b&gt;
 &lt;p&gt;
@@
 <param name="mtCopper" value="0.035mm 0.035mm 0.035mm 0.035mm 0.035mm 0.035mm 0.035mm 0.035mm 0.035mm 0.035mm 0.035mm 0.035mm 0.035mm 0.035mm 0.035mm 0.035mm"/>
 <param name="mtIsolate" value="1.5mm 0.15mm 0.2mm 0.15mm 0.2mm 0.15mm 0.2mm 0.15mm 0.2mm 0.15mm 0.2mm 0.15mm 0.2mm 0.15mm 0.2mm"/>
-<param name="mdWireWire" value="8mil"/>
-<param name="mdWirePad" value="8mil"/>
-<param name="mdWireVia" value="8mil"/>
-<param name="mdPadPad" value="8mil"/>
-<param name="mdPadVia" value="8mil"/>
-<param name="mdViaVia" value="8mil"/>
-<param name="mdSmdPad" value="8mil"/>
-<param name="mdSmdVia" value="8mil"/>
-<param name="mdSmdSmd" value="8mil"/>
+<param name="mdWireWire" value="5mil"/>
+<param name="mdWirePad" value="5mil"/>
+<param name="mdWireVia" value="5mil"/>
+<param name="mdPadPad" value="5mil"/>
+<param name="mdPadVia" value="5mil"/>
+<param name="mdViaVia" value="5mil"/>
+<param name="mdSmdPad" value="5mil"/>
+<param name="mdSmdVia" value="5mil"/>
+<param name="mdSmdSmd" value="5mil"/>
 <param name="mdViaViaSameLayer" value="8mil"/>
 <param name="mnLayersViaInSmd" value="2"/>
@@
 <param name="mdSmdStop" value="0mil"/>
 <param name="msWidth" value="10mil"/>
-<param name="msDrill" value="24mil"/>
+<param name="msDrill" value="19mil"/>
 <param name="msMicroVia" value="9.99mm"/>
 <param name="msBlindViaRatio" value="0.5"/>
@@
 <element name="LED1" library="adafruit" package="LED5MMRGB" value="RGBLED_CA-5MM" x="51.9684" y="13.4112"/>
 <element name="LED2" library="adafruit" package="LED5MMRGB" value="RGBLED_CA-5MM" x="51.816" y="36.4236"/>
+<element name="C1" library="SparkFun-Passives" package="0805" value="" x="83.82" y="54.61" rot="R180"/>
 </elements>
 <signals>
@@
 <wire x1="83.4136" y1="32.1564" x2="83.4136" y2="32.3088" width="0.3048" layer="16"/>
 <wire x1="83.4136" y1="32.3088" x2="83.1088" y2="32.6136" width="0.3048" layer="16"/>
+<contactref element="C1" pad="2"/>
+<wire x1="82.92" y1="54.61" x2="82.92" y2="54.8496" width="0.3048" layer="1"/>
+<wire x1="82.92" y1="54.8496" x2="82.1436" y2="55.626" width="0.3048" layer="1"/>
+<wire x1="82.1436" y1="55.626" x2="75.7936" y2="55.626" width="0.3048" layer="1"/>
+<wire x1="75.7936" y1="55.626" x2="74.9046" y2="54.737" width="0.3048" layer="1"/>
 </signal>
 <signal name="+3V3">
@@
 <wire x1="86.174" y1="24.8452" x2="81.8348" y2="24.8452" width="0.3048" layer="1"/>
 <wire x1="81.8348" y1="24.8452" x2="81.28" y2="25.4" width="0.3048" layer="1"/>
+<contactref element="C1" pad="1"/>
 </signal>
 <signal name="+5V">
@@
 <wire x1="19.8628" y1="22.0472" x2="19.8628" y2="13.8176" width="0.254" layer="1"/>
 <wire x1="19.8628" y1="13.8176" x2="22.606" y2="11.0744" width="0.254" layer="1"/>
-<wire x1="22.606" y1="11.0744" x2="25.3492" y2="11.0744" width="0.254" layer="1"/>
-<wire x1="25.3492" y1="11.0744" x2="33.8836" y2="19.6088" width="0.254" layer="1"/>
-<wire x1="33.8836" y1="19.6088" x2="33.8836" y2="23.2664" width="0.254" layer="1"/>
+<wire x1="22.606" y1="11.0744" x2="25.1968" y2="11.0744" width="0.254" layer="1"/>
+<wire x1="25.1968" y1="11.0744" x2="33.8836" y2="19.7612" width="0.254" layer="1"/>
+<wire x1="33.8836" y1="19.7612" x2="33.8836" y2="23.2664" width="0.254" layer="1"/>
 <wire x1="33.8836" y1="23.2664" x2="33.0012" y2="23.2664" width="0.254" layer="1"/>
 <wire x1="33.0012" y1="23.2664" x2="32.8848" y2="23.15" width="0.254" layer="1"/>
