File: RGBClock.sch (EAGLE design)
At the start: 31 parts, among them K1 PIN20X2

Commit message: Finished board
Parts:
- removed D1, D2: LED-RGB-CA-THRUDIFFUSE, SparkFun-LED:LED-RGB-CA-THRUDIFFUSE
- removed R10, R11, R12, R13, R14, R15, R16, R17, R18, R7, R8, R9: (no value), SparkFun-Passives:RESISTOR0805-RES
- added LED1, LED2: RGBLED_CA-5MM, adafruit:RGBLED_CA-5MM
Connections:
- removed net N$6: D1.BLUE_CATHODE, D2.BLUE_CATHODE, U$8.BLUE8
- new net N$3: LED1.BLUE, LED2.BLUE, U$8.BLUE8
- net +3V3: now also U$6.VCC, U$7.VCC, U$8.VCC, U$9.VCC; no longer R10.2, R11.2, R12.2, R13.2, R14.2, R15.2, R16.2, R17.2, R18.2, R7.2, R8.2, R9.2
- net +5V: now also LED1.VCC, LED2.VCC, U$2.17, U$3.17, U$4.17, U$5.17
- net /BOE: no longer R12.1, R15.1, R18.1, R9.1
- net /GOE: no longer R11.1, R14.1, R17.1, R8.1
- net /ROE: no longer R10.1, R13.1, R16.1, R7.1
- net N$2: now also LED1.RED, LED2.RED; no longer D1.RED_CATHODE, D2.RED_CATHODE
- net N$5: now also LED1.GREEN, LED2.GREEN; no longer D1.GREEN_CATHODE, D2.GREEN_CATHODE

Commit message: Board, gerbers, and BOM
Parts:
- added C1: (no value), SparkFun-Passives:CAP0805
Connections:
- net +3V3: now also C1.1
- net GND: now also C1.2
Changed lines of the file:
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@@
 <part name="LED1" library="adafruit" deviceset="RGBLED_CA" device="-5MM"/>
 <part name="LED2" library="adafruit" deviceset="RGBLED_CA" device="-5MM"/>
+<part name="C1" library="SparkFun-Passives" deviceset="CAP" device="0805"/>
 </parts>
 <sheets>
@@
 <instance part="LED1" gate="G$1" x="342.9" y="83.82"/>
 <instance part="LED2" gate="G$1" x="342.9" y="104.14"/>
+<instance part="C1" gate="G$1" x="0" y="195.58"/>
 </instances>
 <busses>
@@
 <wire x1="40.64" y1="185.42" x2="53.34" y2="185.42" width="0.1524" layer="91"/>
 <junction x="53.34" y="185.42"/>
+<pinref part="C1" gate="G$1" pin="2"/>
+<wire x1="0" y1="193.04" x2="0" y2="185.42" width="0.1524" layer="91"/>
+<wire x1="0" y1="185.42" x2="40.64" y2="185.42" width="0.1524" layer="91"/>
+<junction x="40.64" y="185.42"/>
 </segment>
 </net>
@@
 <wire x1="10.16" y1="195.58" x2="10.16" y2="200.66" width="0.1524" layer="91"/>
 <junction x="10.16" y="200.66"/>
-</segment>
-<segment>
+<pinref part="C1" gate="G$1" pin="1"/>
+<wire x1="10.16" y1="200.66" x2="0" y2="200.66" width="0.1524" layer="91"/>
+</segment>
+<segment>
