File: MicroVersion.sch (EAGLE design)
At the start: 12 parts, among them IC1 MEGA8-AI, Y1 16MHz

Commit message: More microcontroller version
Parts:
- removed IC1: MEGA8-AI, atmel:MEGA8-AI
- removed Y1: 16MHz, SparkFun-FreqCtrl:CRYSTALSMD
- added JP1: POWER_JACKPTH, SparkFun-Connectors:POWER_JACKPTH
- added JP2: FTDI_DEVICE, SparkFun-Connectors:FTDI_DEVICE
- added LED1, LED2: RGBLED_CA-5MM, adafruit:RGBLED_CA-5MM
- added Q1: (no value), adafruit:CRYSTALCTS406
- added U$1, U$2, U$3, U$4: RGBSEVENSEGMENT, Benchoff:RGBSEVENSEGMENT
- added U$5, U$6, U$7, U$8: LED2472G, Benchoff:LED2472G
- added U2: (no value), SparkFun-PowerIC:V_REG_78XXSIDE
- added U4: ATMEGA328P_TQFP, SparkFun-DigitalIC:ATMEGA328P_TQFP
Connections:
- removed net +3V3: C4.1, R4.2, R5.2, RTC1.RST, RTC1.VCC
- new net VCC: C1.2, C4.1, ISP1.VCC, JP2.VCC, R4.2, R5.2, RTC1.RST, RTC1.VCC, U2.OUT, U4.VCC@4, U4.VCC@6
- net CLOCK: now also U4.PD7(AIN1); no longer IC1.PD7(AIN1)
- net DATA: now also U4.PD2(INT0); no longer IC1.PD2(INT0)
- net GND: now also JP1.PWR, JP2.GND, U2.GND, U4.AGND, U4.AVCC, U4.GND@3, U4.GND@5; no longer IC1.GND, IC1.GND@1, IC1.GND@2
- net LATCH: now also U4.PD4(XCK/T0); no longer IC1.PD4(XCK/T0)
- net MISO: now also U4.PB4(MISO); no longer IC1.PB4(MISO)
- net MOSI: now also U4.PB3(MOSI/OC2); no longer IC1.PB3(MOSI/OC2)
- net N$2: now also U4.PD3(INT1); no longer IC1.PD3(INT1)
- net N$3: now also U4.PD5(T1); no longer IC1.PD5(T1)
- net N$4: now also U4.PD6(AIN0); no longer IC1.PD6(AIN0)
- net N$5: now also JP1.GND, JP1.GNDBREAK, U2.IN; no longer C1.2, IC1.AVCC, IC1.VCC@1, IC1.VCC@2, ISP1.VCC
- net RESET: now also U4.PC6(/RESET); no longer IC1.PC6(/RESET)
- net SCK: now also U4.PB5(SCK); no longer IC1.PB5(SCK)
- net SCL: now also U4.PC5(ADC5/SCL); no longer IC1.PC5(ADC5/SCL)
- net SDA: now also U4.PC4(ADC4/SDA); no longer IC1.PC4(ADC4/SDA)
- net XTAL1: now also Q1.2, U4.PB6(XTAL1/TOSC1); no longer IC1.PB6(XTAL1/TOSC1), Y1.2
- net XTAL2: now also Q1.1, U4.PB7(XTAL2/TOSC2); no longer IC1.PB7(XTAL2/TOSC2), Y1.1
Other:
- moved on the sheet: C2, C3
