File: MicroVersion.brd (EAGLE design)
At the start: 116.8 x 49.5 mm, 25 parts, among them U4 ATMEGA328P_TQFP

Commit message: Huge update to micro version
Parts:
- removed C1: 100n, SparkFun-Passives:0805
- removed S1: SWITCH-MOMENTARY-2SMD, SparkFun-Electromechanical:TACTILE-SWITCH-SMD
- removed U2: (no value), SparkFun-PowerIC:78XXL
- added C5: 0.47uF, SparkFun-Capacitors:EIA3216
- added C6: 22uF, SparkFun-Capacitors:1210
- added IC1: 7805DT, linear:TO252
- added IC2: REG1117, burr-brown:SOT223
- added R1, R2: 10k, SparkFun-Passives:0805
- added R10, R11, R12, R13, R14, R15, R16, R17, R18, R19, R20, R21, R22, R3, R6, R7, R8, R9: (no value), SparkFun-Passives:0805
- added S2, S3, S4: SWITCH-MOMENTARY-2SMD-1101NE, SparkFun-Electromechanical:TACTILE-SWITCH-1101NE
- added U$10: ESP8266-03, #ESP8266:ESP-03
- added U1: TSX0102, adafruit:VFSOP-8
- moved BAT1 61.4 mm to (120.2, 13.6), flipped to the bottom
- moved R5 55.8 mm to (90.8, 22.5)
- moved R4 55.8 mm to (90.8, 19.3)
- moved C4 51.0 mm to (87.4, 18.6), turned to 270 degrees
- moved JP1 45.3 mm to (151.2, 17.4), flipped to the bottom, turned to 270 degrees
- moved U$7 44.5 mm to (108.3, 40.3), turned to 90 degrees
- moved U$8 44.5 mm to (132.4, 40.3), turned to 90 degrees
- moved U$6 44.3 mm to (77.5, 40.3), turned to 90 degrees
- moved U$4 44.2 mm to (120.7, 22.5)
- moved U$2 44.2 mm to (66.0, 22.5)
- moved U$3 44.2 mm to (96.5, 22.5)
- moved U$1 43.9 mm to (41.6, 22.5)
- moved U$5 43.9 mm to (53.0, 40.3), turned to 90 degrees
- moved JP2 43.9 mm to (37.5, 22.2), flipped to the bottom
- moved LED1 43.9 mm to (92.7, 48.3)
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Connections:
- new net /BOE: U$5.32, U$6.32, U4.10
- new net /GOE: U$5.33, U$6.33, U4.9
- new net /ROE: U$5.34, U$6.34, U4.1
- new net 1BLUE1: U$1.24, U$5.15
- new net 1BLUE2: U$1.21, U$5.18
- new net 1BLUE3: U$1.19, U$5.21
- new net 1BLUE4: U$1.18, U$5.24
- new net 1BLUE5: U$1.9, U$5.37
- new net 1BLUE6: U$1.2, U$5.40
- new net 1BLUE7: U$1.5, U$5.43
- new net 1GREEN1: U$1.16, U$5.14
- new net 1GREEN2: U$1.22, U$5.17
- new net 1GREEN3: U$1.15, U$5.20
- new net 1GREEN4: U$1.13, U$5.23
- new net 1GREEN5: U$1.1, U$5.38
- new net 1GREEN6: U$1.3, U$5.41
- new net 1GREEN7: U$1.11, U$5.44
- new net 1RED1: U$1.25, U$5.13
- new net 1RED2: U$1.23, U$5.16
- new net 1RED3: U$1.20, U$5.19
- new net 1RED4: U$1.14, U$5.22
- new net 1RED5: U$1.10, U$5.39
- new net 1RED6: U$1.4, U$5.42
- new net 1RED7: U$1.6, U$5.45
- new net N$11: U$10.URXD, U1.P$5
- new net N$12: U$10.UTXD, U1.P$4
- new net N$7: R22.2, S3.1, U4.26
- new net N$8: R21.1, S2.1, U4.25
- new net N$9: IC2.2, U$10.VCC, U1.P$3, U1.P$6
- new net RXD: JP2.P$3, U4.30
- new net TXD: JP2.P$2, U4.31
- net CLOCK: now also R1.1, U$5.4, U$6.4, U$7.4, U$8.4, U4.13; no longer U4.11
- net DATA: now also R2.1, U$5.2, U4.12; no longer U4.32
- net GND: now also C5.C, C6.1, IC1.3, IC2.1, JP2.P$5, S2.2, S3.2, S4.2, U$10.GND, U1.P$2; no longer C1.1, S1.3, U2.GND
- net LATCH: now also U$5.3, U$6.3, U$7.3, U$8.3, U4.14; no longer U4.2
- net N$2: now also U$5.35, U$6.2; no longer U4.1
- net N$3: now also U$6.35, U$7.2; no longer U4.9
- net N$4: now also U$7.35, U$8.2; no longer U4.10
- net N$5: now also C5.A, IC1.1; no longer U2.IN
- net RESET: now also JP2.P$1, S4.1; no longer S1.1
- net VCC: now also C6.2, IC1.2, IC2.3, R1.2, R2.2, R21.2, R22.1, U1.P$7; no longer C1.2, U2.OUT
Routing:
- net LATCH: track 0.00 -> 171.2 mm, vias 0 -> 5
- net CLOCK: track 0.00 -> 159.2 mm, vias 0 -> 5
- net N$3: track 0.00 -> 60.4 mm, vias 0 -> 2
- net DATA: track 0.00 -> 54.5 mm, vias 0 -> 2
- net N$2: track 0.00 -> 51.4 mm, vias 0 -> 2
- net N$4: track 0.00 -> 50.3 mm, vias 0 -> 2
- net /ROE: track 0.00 -> 44.5 mm, vias 0 -> 2
- net /BOE: track 0.00 -> 40.5 mm
- net TXD: track 0.00 -> 39.7 mm, vias 0 -> 1
- net N$9: track 0.00 -> 38.7 mm
- net /GOE: track 0.00 -> 37.7 mm
- net RXD: track 0.00 -> 37.0 mm, vias 0 -> 1
- net N$1: track 14.8 -> 46.0 mm, vias 0 -> 1
- net XTAL2: track 36.0 -> 11.6 mm
- net XTAL1: track 37.2 -> 14.5 mm
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Other:
- board text added: "Hour"
- board text added: "Minute"
- board text added: "RESET"
- board text added: "Use CR1225 3V Lithium"

Commit message: Update
Parts:
- removed R10, R11, R12, R13, R14, R15, R16, R17, R18, R19, R20, R3, R6, R7, R8, R9: (no value), SparkFun-Passives:0805
Changed lines of the file:
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@@
 <layer number="14" name="Route14" color="1" fill="6" visible="no" active="no"/>
 <layer number="15" name="Route15" color="4" fill="6" visible="no" active="no"/>
-<layer number="16" name="Bottom" color="1" fill="1" visible="yes" active="yes"/>
+<layer number="16" name="Bottom" color="1" fill="1" visible="no" active="yes"/>
 <layer number="17" name="Pads" color="2" fill="1" visible="yes" active="yes"/>
 <layer number="18" name="Vias" color="2" fill="1" visible="yes" active="yes"/>
 <layer number="19" name="Unrouted" color="6" fill="1" visible="yes" active="yes"/>
 <layer number="20" name="Dimension" color="15" fill="1" visible="yes" active="yes"/>
-<layer number="21" name="tPlace" color="7" fill="1" visible="yes" active="yes"/>
+<layer number="21" name="tPlace" color="7" fill="1" visible="no" active="yes"/>
 <layer number="22" name="bPlace" color="7" fill="1" visible="yes" active="yes"/>
 <layer number="23" name="tOrigins" color="15" fill="1" visible="yes" active="yes"/>
@@
 <element name="R1" library="SparkFun-Passives" package="0805" value="10k" x="39.17315" y="32.04845" rot="R180"/>
 <element name="R2" library="SparkFun-Passives" package="0805" value="10k" x="40.132" y="34.44875" rot="R180"/>
-<element name="R3" library="SparkFun-Passives" package="0805" value="" x="-38.1" y="-8.89"/>
-<element name="R6" library="SparkFun-Passives" package="0805" value="" x="-41.91" y="-8.89"/>
-<element name="R7" library="SparkFun-Passives" package="0805" value="" x="-45.72" y="-8.89"/>
-<element name="R8" library="SparkFun-Passives" package="0805" value="" x="-49.53" y="-8.89"/>
-<element name="R9" library="SparkFun-Passives" package="0805" value="" x="-53.34" y="-8.89"/>
-<element name="R10" library="SparkFun-Passives" package="0805" value="" x="-57.15" y="-8.89"/>
-<element name="R11" library="SparkFun-Passives" package="0805" value="" x="-60.96" y="-8.89"/>
-<element name="R12" library="SparkFun-Passives" package="0805" value="" x="-64.77" y="-8.89"/>
-<element name="R13" library="SparkFun-Passives" package="0805" value="" x="-68.58" y="-8.89"/>
-<element name="R14" library="SparkFun-Passives" package="0805" value="" x="-72.39" y="-8.89"/>
-<element name="R15" library="SparkFun-Passives" package="0805" value="" x="-76.2" y="-8.89"/>
-<element name="R16" library="SparkFun-Passives" package="0805" value="" x="-80.01" y="-8.89"/>
-<element name="R17" library="SparkFun-Passives" package="0805" value="" x="-83.82" y="-8.89"/>
-<element name="R18" library="SparkFun-Passives" package="0805" value="" x="-87.63" y="-8.89"/>
-<element name="R19" library="SparkFun-Passives" package="0805" value="" x="-91.44" y="-8.89"/>
-<element name="R20" library="SparkFun-Passives" package="0805" value="" x="-95.25" y="-8.89"/>
 <element name="S2" library="SparkFun-Electromechanical" package="TACTILE-SWITCH-1101NE" value="SWITCH-MOMENTARY-2SMD-1101NE" x="81.28" y="10.16">
 <attribute name="PROD_ID" value="SWCH-00815" x="81.28" y="10.16" size="1.778" layer="27" display="off"/>
